File: hardware/Communication Board/Communication Board.kicad_sch (KiCad schematic)
At the start: 17 parts, among them J1 CC1101, Q1 IRLZ44N, U1 STM32F411CEUx, U2 LM358

Commit message: finished ground station board. started communication board.
Parts:
- removed C4: 100n, symbol Device:C
- removed Q1: IRLZ44N, Package_TO_SOT_THT:TO-220-3_Vertical, symbol Transistor_FET:IRLZ44N
- removed R3: 1k, symbol Device:R_US
- removed U2: LM358, symbol Amplifier_Operational:LM358
- added C5: 10u, symbol Device:C_US
- added C6: 100n, symbol Device:C
- added Q1: 2N2222, symbol Simulation_SPICE:NPN
- added R3: 20k, symbol Device:R_Variable_US
- added R7: 47k, symbol Device:R_US
- added R8, R9: 10k, symbol Device:R_US
- added U2, U3: MCP6022, symbol Amplifier_Operational:MCP6022
- C3: value 22p -> 5p
- D3: value 3W_IR_LED -> TSAL6200_IRLED
- R2: value 470k -> 1k
- R4: value 5 -> 10
Connections:
- net +3.3V: now also C5.1, R7.2
- net GNDREF: now also C5.2, Q1.3 (E), R8.1, R9.1, U2.3 (+)
- net IR_LED_OUT: no longer U1.19 (PB1)
- net TIA_OUT: now also C6.2; no longer U1.18 (PB0)
- net at R5.2, R6.2: now also Q1.2 (B)
- net at D3.1 (K): now also Q1.1 (C)
- net at C3.1, D2.1 (K), R2.1: now also U2.2 (-)
- net at C3.2: now also R3.2, U2.1; no longer R2.2
- new net: C6.1, R9.2, U3.2 (-)
- new net: R7.1, R8.2, U3.3 (+)
- new net: R2.2, R3.1
- new net IrDA RX: U3.1
Other:
- note added: "10 ohm for higher power output and longer range"
- note added: "2N2222 has faster switching speed."
- note removed: "This will pull 0.5A when driven at full duty cycle. Be careful drawing this power from Black Pill board."
- moved on the sheet: C1, C2, C3, D1, D2, D3, J1, R1, R4, R5, R6, U1
