File: hardware/Electrical/Communication Board/Communication Board.kicad_sch (KiCad schematic)
At the start: 22 parts, among them J1 CC1101, Q1 2N2222, U1 STM32F411CEUx, U2 MCP6022, U3 MCP6022

Commit message: too much
Parts:
- added C4: 100n, symbol Device:C
- added R10, R11: 10k, symbol Device:R_US
Connections:
- net +3.3V: now also R10.2
- net GNDREF: now also C4.1, R11.1; no longer U2.3 (+)
- new net: C4.2, R10.1, R11.2
Other:
- note removed: "Transimpedance amplifier to turn photodiode's small current into a sensible voltage."
